File: OpenAmigaVideoHybrid.kicad_pcb (KiCad board)
At the start: 2 copper layers, 56.4 x 21.1 mm, 52 parts, among them J1 Conn_01x22, J99 OSHW_LOGO, Q1 2N3904, Q2 2N3904, Q3 2N3904, Q4 2N3904, Q5 2N3904, Q6 2N3906

Commit message: Modify PCB and add production files
Parts:
- C5, Q5, Q6, R30, R31, R32, R33, R34, R35, R36, R37, R38, R39: moved to B.Cu
- moved C3 9.80 mm to (161.8, 106.2), turned to 0 degrees
- moved R36 9.69 mm to (150.5, 106.8), turned to 0 degrees
- moved Q5 9.47 mm to (153.4, 110.9)
- moved R37 7.03 mm to (170.9, 119.1)
- moved R35 6.64 mm to (145.5, 106.8), turned to 0 degrees
- moved Q6 5.51 mm to (170.9, 115.2)
- moved R30 5.39 mm to (155.3, 107.1), turned to 180 degrees
- moved C5 4.16 mm to (168.5, 106.2), turned to 180 degrees
- moved R34 4.11 mm to (148.5, 110.5), turned to -90 degrees
- moved C2 3.28 mm to (137.8, 106.3), turned to 180 degrees
- moved R39 2.18 mm to (167.6, 121.7)
- moved R32 1.91 mm to (135.5, 110.4)
- moved R33 1.89 mm to (140.8, 110.5)
- moved R38 1.78 mm to (166.4, 115.1)
- moved R31 1.52 mm to (161.0, 118.4)
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Routing:
- net GND: track 160.8 -> 46.8 mm, vias 26 -> 17
- net VCC: track 159.2 -> 129.9 mm, vias 0 -> 2
- net Net-(Q5-Pad1): track 6.75 -> 29.2 mm, vias 0 -> 2
- net Net-(Q5-Pad2): track 36.1 -> 54.8 mm
- net Net-(Q5-Pad3): track 20.6 -> 28.1 mm, vias 0 -> 2
- net Net-(Q6-Pad3): track 13.4 -> 7.35 mm
- net Net-(Q3-Pad2): track 30.5 -> 24.8 mm, vias 1 -> 0
- net /csync: track 9.24 -> 6.40 mm
- net Net-(Q1-Pad2): track 26.2 -> 24.4 mm, vias 1 -> 0
- net Net-(Q2-Pad2): track 25.7 -> 27.3 mm, vias 1 -> 0
- net /comp: track 4.61 -> 3.29 mm
- net Net-(Q4-Pad1): track 10.8 -> 9.98 mm
- net Net-(Q4-Pad2): track 15.1 -> 14.4 mm
- net Net-(Q1-Pad1): track 7.13 -> 6.43 mm
- net /blue: track 4.49 -> 5.17 mm
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Other:
- net class Default removed
- net class Power removed
- board text added: "github.com/SukkoPera/OpenAmigaVideoHybrid Single-layer PCB by PHL"
- board text removed: "github.com/SukkoPera/OpenAmigaVideoHybrid"
